File: tps61021a-slim.kicad_pcb (KiCad board)
At the start: 2 copper layers, 15.7 x 15.7 mm, 9 parts, among them J1 Conn_01x04_Male, U1 TPS61021A

Commit message: routed completed
Parts:
- added REF**: OSHW-Symbol_6.7x6mm_SilkScreen, Symbol:OSHW-Symbol_6.7x6mm_SilkScreen, B.Cu at (112.3, 103.6)
- moved C2 10.7 mm to (102.6, 105.3), turned to 180 degrees
- moved C1 10.7 mm to (113.3, 109.1)
- moved L1 9.33 mm to (112.4, 103.6), turned to 180 degrees
- moved R2 7.85 mm to (102.6, 109.1)
- moved C4 6.26 mm to (107.2, 105.3)
- moved C3 6.10 mm to (107.2, 101.6)
- moved R1 6.10 mm to (102.6, 101.6), turned to 180 degrees
Routing:
- net Earth: track 0.00 -> 24.3 mm
- net Net-(C2-Pad1): track 0.00 -> 19.3 mm, vias 0 -> 2
- net Net-(C1-Pad1): track 0.00 -> 18.7 mm, vias 0 -> 1
- net Net-(C2-Pad2): track 0.00 -> 15.2 mm
- net Net-(L1-Pad2): track 0.00 -> 11.1 mm, vias 0 -> 2
- net Net-(J1-Pad1): track 0.00 -> 5.10 mm
- added copper zone on B.Cu, net Earth
- added copper zone on F.Cu, net Earth
Other:
- board text added: "CE"
- board text added: "GND"
- board text added: "TPS61021"
- board text added: "VIN"
- board text added: "VOUT"
